File: PCB/Modules/Buck12v-5v-TPS561208/Buck12v-5v-TPS561208.kicad_pcb (KiCad board)
At the start: 2 copper layers, 42.7 x 25.2 mm, 8 parts, among them U1 TPS561208DDCT

Commit message: Small new changes
Signed-off-by: Simonca Raul <simonca.raul@gmail.com>
Parts:
- moved Rfbt1 11.0 mm to (155.7, 92.3), turned to 180 degrees
- moved Cout1 8.80 mm to (162.2, 86.9), turned to -90 degrees
- moved U1 8.32 mm to (146.9, 87.2)
- moved L1 6.23 mm to (155.4, 86.5), turned to 180 degrees
- moved Rfbb1 5.68 mm to (147.0, 90.6), turned to 180 degrees
- moved Cbst1 5.54 mm to (147.1, 83.6), turned to 180 degrees
- moved Cin2 4.48 mm to (142.6, 87.2), turned to 90 degrees
- moved Cin1 2.41 mm to (139.5, 87.2), turned to 90 degrees
Connections:
- net Net-(U1-SW) renamed /SW
- net Net-(U1-VBST) renamed /VBST
- net Net-(U1-VFB) renamed /VFB
Routing:
- net GND: track 0.00 -> 28.0 mm
- net /SW: track 0.00 -> 22.2 mm, vias 0 -> 2
- net /VFB: track 0.00 -> 10.7 mm
- net +12V: track 0.00 -> 9.71 mm
- net +5V: track 0.00 -> 5.83 mm
- net /VBST: track 0.00 -> 2.93 mm
