File: PCB/Modules/Buck12v-5v-TPS561208/Buck12v-5v-TPS561208.kicad_pcb (KiCad board)
At the start: 2 copper layers, 42.7 x 25.2 mm, 8 parts, among them U1 TPS561208DDCT

Commit message: Test kicad
Signed-off-by: Simonca Raul <simonca.raul@gmail.com>
Parts:
- moved Rfbt1 9.07 mm to (146.8, 90.5)
- moved Rfbb1 5.26 mm to (151.1, 87.3), turned to 90 degrees
- moved Cout1 2.00 mm to (164.2, 86.8), turned to 90 degrees
- moved L1 1.76 mm to (157.2, 86.7)
- turned Cbst1 to 0 degrees
Routing:
- net +5V: track 5.83 -> 18.2 mm
- net GND: track 28.0 -> 34.2 mm
- net /VFB: track 10.7 -> 7.09 mm
- net /SW: track 22.2 -> 19.0 mm
- net /VBST: track 2.93 -> 4.33 mm
