File: PCB/Modules/Buck12v-5v-TPS561208/Buck12v-5v-TPS561208.kicad_sch (KiCad schematic)
At the start: 8 parts, among them U1 TPS561208DDCT

Commit message: Small new changes
Signed-off-by: Simonca Raul <simonca.raul@gmail.com>
Connections:
- net +12V: now also Rfbb1.1, Rfbt1.2, U1.4 (VFB)
- net SW: now reaches Cbst1.2, L1.1, U1.2 (SW)
- net VBST: now reaches Cbst1.1, U1.6 (VBST)
Changed lines of the file:
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@@
-	(wire
-		(pts
-			(xy 133.35 83.82) (xy 129.54 83.82)
-		)
-		(stroke
-			(width 0)
-			(type default)
-		)
-	)
 	(wire
 		(pts
@@
 	(wire
 		(pts
+			(xy 129.54 83.82) (xy 133.35 83.82)
+		)
+		(stroke
+			(width 0)
+			(type default)
+		)
+	)
+	(wire
+		(pts
 			(xy 132.08 86.36) (xy 132.08 102.87)
 		)
@@
 		)
 	)
+	(label "EN"
+		(at 132.08 83.82 0)
+		(fields_autoplaced yes)
+		(effects
+			(font
+				(size 1.27 1.27)
+			)
+			(justify left bottom)
+		)
+	)
+	(label "VBST"
+		(at 170.18 78.74 0)
+		(fields_autoplaced yes)
+		(effects
+			(font
+				(size 1.27 1.27)
+			)
+			(justify left bottom)
+		)
+	)
+	(label "VFB"
+		(at 132.08 86.36 0)
+		(fields_autoplaced yes)
+		(effects
+			(font
+				(size 1.27 1.27)
+			)
+			(justify left bottom)
+		)
+	)
+	(label "SW"
+		(at 133.35 91.44 0)
+		(fields_autoplaced yes)
+		(effects
+			(font
+				(size 1.27 1.27)
+			)
+			(justify left bottom)
+		)
+	)
+	(label "VIN"
+		(at 132.08 88.9 0)
+		(fields_autoplaced yes)
+		(effects
+			(font
+				(size 1.27 1.27)
+			)
+			(justify left bottom)
+		)
+	)
